File: EdiabasLib/EnetAdapter/Layout/AdapterBoard/ObdBackplane.sch (EAGLE design)
At the start: 10 parts

Commit message: Added new solder pad
Parts:
- added P'-: SE14, solpad:SE14
- P+: value 5V -> SE14; device pinhead:PINHD-1X1_2.54 -> solpad:SE14
- P-: value GND -> SE14; device pinhead:PINHD-1X1_2.54 -> solpad:SE14
Connections:
- new net GND2: IN-.1, P'-.MP
- net +5V: now also P+.MP; no longer P+.1
- net GND: now also P-.MP; no longer P-.1
Changed lines of the file:
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@@
 <part name="OUT-" library="pinhead" deviceset="PINHD-1X1" device="_2.54" value="GND"/>
 <part name="P+2" library="supply1" deviceset="+5V" device=""/>
-<part name="P+" library="pinhead" deviceset="PINHD-1X1" device="_2.54" value="5V"/>
-<part name="P-" library="pinhead" deviceset="PINHD-1X1" device="_2.54" value="GND"/>
 <part name="JP1" library="obd_special" deviceset="PINHD-1X8" device="_1.00" value="ETHERNET"/>
+<part name="P+" library="solpad" deviceset="SE14" device=""/>
+<part name="P-" library="solpad" deviceset="SE14" device=""/>
+<part name="P'-" library="solpad" deviceset="SE14" device=""/>
 </parts>
 <sheets>
@@
 <instance part="OUT-" gate="G$1" x="91.44" y="170.18"/>
 <instance part="P+2" gate="1" x="60.96" y="175.26"/>
-<instance part="P+" gate="G$1" x="73.66" y="149.86"/>
-<instance part="P-" gate="G$1" x="91.44" y="149.86"/>
 <instance part="JP1" gate="A" x="-7.62" y="266.7" rot="R90"/>
+<instance part="P+" gate="1" x="71.12" y="152.4"/>
+<instance part="P-" gate="1" x="88.9" y="152.4"/>
+<instance part="P'-" gate="1" x="88.9" y="193.04"/>
 </instances>
 <busses>
@@
 <wire x1="88.9" y1="170.18" x2="88.9" y2="149.86" width="0.1524" layer="91"/>
 <junction x="88.9" y="170.18"/>
-<pinref part="P-" gate="G$1" pin="1"/>
+<pinref part="P-" gate="1" pin="MP"/>
 </segment>
 </net>
@@
 <wire x1="71.12" y1="170.18" x2="71.12" y2="149.86" width="0.1524" layer="91"/>
 <junction x="71.12" y="170.18"/>
-<pinref part="P+" gate="G$1" pin="1"/>
+<pinref part="P+" gate="1" pin="MP"/>
 </segment>
 </net>
@@
 </segment>
 </net>
+<net name="GND2" class="0">
+<segment>
+<pinref part="IN-" gate="G$1" pin="1"/>
+<pinref part="P'-" gate="1" pin="MP"/>
+<wire x1="88.9" y1="210.82" x2="88.9" y2="190.5" width="0.1524" layer="91"/>
+</segment>
+</net>

Commit message: Library update
Parts:
- IN+, IN-, OUT+, OUT-: device pinhead:PINHD-1X1_2.54 -> pinhead:PINHD-1X1
Changed lines of the file:
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@@
 <part name="GND1" library="supply1" deviceset="GND" device=""/>
 <part name="P+1" library="supply1" deviceset="+12V" device=""/>
-<part name="IN+" library="pinhead" deviceset="PINHD-1X1" device="_2.54" value="12V"/>
-<part name="IN-" library="pinhead" deviceset="PINHD-1X1" device="_2.54" value="GND"/>
-<part name="OUT+" library="pinhead" deviceset="PINHD-1X1" device="_2.54" value="5V"/>
-<part name="OUT-" library="pinhead" deviceset="PINHD-1X1" device="_2.54" value="GND"/>
+<part name="IN+" library="pinhead" deviceset="PINHD-1X1" device="" value="12V"/>
+<part name="IN-" library="pinhead" deviceset="PINHD-1X1" device="" value="GND"/>
+<part name="OUT+" library="pinhead" deviceset="PINHD-1X1" device="" value="5V"/>
+<part name="OUT-" library="pinhead" deviceset="PINHD-1X1" device="" value="GND"/>
 <part name="P+2" library="supply1" deviceset="+5V" device=""/>
 <part name="JP1" library="obd_special" deviceset="PINHD-1X8" device="_1.00" value="ETHERNET"/>

Commit message: Updated to eagle 8.3.2
Parts:
- D1: value (none) -> 100V
Changed lines of the file:
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@@
 <?xml version="1.0" encoding="utf-8"?>
 <!DOCTYPE eagle SYSTEM "eagle.dtd">
-<eagle version="7.7.0">
+<eagle version="8.3.2">
 <drawing>
 <settings>
 <setting alwaysvectorfont="no"/>
+<setting keepoldvectorfont="yes"/>
 <setting verticaltext="up"/>
 </settings>
@@
 <layer number="230" name="230bmp" color="7" fill="1" visible="yes" active="yes"/>
 <layer number="231" name="231bmp" color="7" fill="1" visible="yes" active="yes"/>
+<layer number="232" name="Eagle3D_PG2" color="7" fill="1" visible="yes" active="yes"/>
+<layer number="233" name="Eagle3D_PG3" color="7" fill="1" visible="yes" active="yes"/>
 <layer number="248" name="Housing" color="7" fill="1" visible="yes" active="yes"/>
 <layer number="249" name="Edge" color="7" fill="1" visible="yes" active="yes"/>
@@
 </classes>
 <parts>
-<part name="OBDII" library="SparkFun-Connectors" deviceset="OBDII" device=""/>
-<part name="D1" library="diode" deviceset="DIODE-" device="DO214AC"/>
-<part name="R1" library="resistor" deviceset="R-EU_" device="R2512" value="511"/>
-<part name="FRAME1" library="frames" deviceset="DINA4_L" device=""/>
-<part name="GND1" library="supply1" deviceset="GND" device=""/>
-<part name="P+1" library="supply1" deviceset="+12V" device=""/>
-<part name="IN+" library="pinhead" deviceset="PINHD-1X1" device="" value="12V"/>
-<part name="IN-" library="pinhead" deviceset="PINHD-1X1" device="" value="GND"/>
-<part name="OUT+" library="pinhead" deviceset="PINHD-1X1" device="" value="5V"/>
-<part name="OUT-" library="pinhead" deviceset="PINHD-1X1" device="" value="GND"/>
-<part name="P+2" library="supply1" deviceset="+5V" device=""/>
+<part name="OBDII" library="SparkFun-Connectors" library_urn="urn:adsk.eagle:library:513" deviceset="OBDII" device="" package3d_urn="urn:adsk.eagle:package:38217/1"/>
+<part name="D1" library="diode" library_urn="urn:adsk.eagle:library:210" deviceset="DIODE-" device="DO214AC" package3d_urn="urn:adsk.eagle:package:43417/2" value="100V"/>
+<part name="R1" library="resistor" library_urn="urn:adsk.eagle:library:348" deviceset="R-EU_" device="R2512" package3d_urn="urn:adsk.eagle:package:26070/1" value="511"/>
+<part name="FRAME1" library="frames" library_urn="urn:adsk.eagle:library:229" deviceset="DINA4_L" device=""/>
+<part name="GND1" library="supply1" library_urn="urn:adsk.eagle:library:371" deviceset="GND" device=""/>
+<part name="P+1" library="supply1" library_urn="urn:adsk.eagle:library:371" deviceset="+12V" device=""/>
+<part name="IN+" library="pinhead" library_urn="urn:adsk.eagle:library:325" deviceset="PINHD-1X1" device="" package3d_urn="urn:adsk.eagle:package:22485/2" value="12V"/>
+<part name="IN-" library="pinhead" library_urn="urn:adsk.eagle:library:325" deviceset="PINHD-1X1" device="" package3d_urn="urn:adsk.eagle:package:22485/2" value="GND"/>
+<part name="OUT+" library="pinhead" library_urn="urn:adsk.eagle:library:325" deviceset="PINHD-1X1" device="" package3d_urn="urn:adsk.eagle:package:22485/2" value="5V"/>
+<part name="OUT-" library="pinhead" library_urn="urn:adsk.eagle:library:325" deviceset="PINHD-1X1" device="" package3d_urn="urn:adsk.eagle:package:22485/2" value="GND"/>
+<part name="P+2" library="supply1" library_urn="urn:adsk.eagle:library:371" deviceset="+5V" device=""/>
 <part name="JP1" library="obd_special" deviceset="PINHD-1X8" device="_1.00" value="ETHERNET"/>
-<part name="P+" library="solpad" deviceset="SE14" device=""/>
-<part name="P-" library="solpad" deviceset="SE14" device=""/>
-<part name="P'-" library="solpad" deviceset="SE14" device=""/>
+<part name="P+" library="solpad" library_urn="urn:adsk.eagle:library:364" deviceset="SE14" device="" package3d_urn="urn:adsk.eagle:package:26504/1"/>
+<part name="P-" library="solpad" library_urn="urn:adsk.eagle:library:364" deviceset="SE14" device="" package3d_urn="urn:adsk.eagle:package:26504/1"/>
+<part name="P'-" library="solpad" library_urn="urn:adsk.eagle:library:364" deviceset="SE14" device="" package3d_urn="urn:adsk.eagle:package:26504/1"/>
 </parts>
 <sheets>
@@
 </schematic>
 </drawing>
+<compatibility>
+<note version="8.2" severity="warning">
+Since Version 8.2, EAGLE supports online libraries. The ids
+of those online libraries will not be understood (or retained)
+with this version.
+</note>
+<note version="8.3" severity="warning">
+Since Version 8.3, EAGLE supports URNs for individual library
+assets (packages, symbols, and devices). The URNs of those assets
+will not be understood (or retained) with this version.
+</note>
+<note version="8.3" severity="warning">
+Since Version 8.3, EAGLE supports the association of 3D packages
+with devices in libraries, schematics, and board files. Those 3D
+packages will not be understood (or retained) with this version.
+</note>
+</compatibility>
 </eagle>
